Commit message: Removed all comments

File: box_sim/urdf/box.gazebo.xacro (robot description, xacro)
@@ -1,10 +1,10 @@
 <?xml version="1.0"?>
-<robot xmlns:xacro="http://www.ros.org/wiki/xacro">
-    <!-- Load Gazebo lib and set the robot namespace -->
+<robot
+    xmlns:xacro="http://www.ros.org/wiki/xacro">
     <gazebo>
         <plugin name="gazebo_ros_control" filename="libgazebo_ros_control.so">
-            <robotNamespace>/</robotNamespace>
+            <robotNamespace></robotNamespace>
             <robotSimType>steer_bot_hardware_gazebo/SteerBotHardwareGazebo</robotSimType>
         </plugin>
-  </gazebo>
+    </gazebo>
 </robot>

File: box_sim/urdf/box.transmission.xacro (robot description, xacro)
@@ -1,6 +1,7 @@
 <?xml version="1.0"?>
-<robot xmlns:xacro="http://www.ros.org/wiki/xacro">
-<xacro:macro name="box_transmission">
-       <transmission name="box_tran_1">
+<robot
+    xmlns:xacro="http://www.ros.org/wiki/xacro">
+    <xacro:macro name="box_transmission">
+        <transmission name="box_tran_1">
             <type>transmission_interface/SimpleTransmission</type>
             <joint name="right_steer_joint">
@@ -12,15 +13,4 @@
             </actuator>
         </transmission>
-      <!-->  <transmission name="junior_car_tran_2">
-            <robotNamespace>/junior_car</robotNamespace>
-            <type>transmission_interface/SimpleTransmission</type>
-            <joint name="right_steer_wheel_joint">
-                <hardwareInterface>VelocityJointInterface</hardwareInterface>
-            </joint>
-            <actuator name="junior_car_motor_2">
-                <hardwareInterface>VelocityJointInterface</hardwareInterface>
-                <mechanicalReduction>1</mechanicalReduction>
-            </actuator>
-        </transmission>-->
         <transmission name="box_tran_3">
             <type>transmission_interface/SimpleTransmission</type>
@@ -33,15 +23,4 @@
             </actuator>
         </transmission>
-    <!-->    <transmission name="junior_car_tran_4">
-            <robotNamespace>/junior_car</robotNamespace>
-            <type>transmission_interface/SimpleTransmission</type>
-            <joint name="left_steer_wheel_joint">
-                <hardwareInterface>VelocityJointInterface</hardwareInterface>
-            </joint>
-            <actuator name="junior_car_motor_4">
-                <hardwareInterface>VelocityJointInterface</hardwareInterface>
-                <mechanicalReduction>1</mechanicalReduction>
-            </actuator>
-        </transmission> -->
         <transmission name="box_tran_5">
             <type>transmission_interface/SimpleTransmission</type>
@@ -85,26 +64,4 @@
             </actuator>
         </transmission>
-  <!-->  <transmission name="junior_car_tran_5double">
-            <robotNamespace>/junior_car</robotNamespace>
-            <type>transmission_interface/SimpleTransmission</type>
-            <joint name="right_drive_wheel_joint">
-                <hardwareInterface>VelocityJointInterface</hardwareInterface>
-            </joint>
-            <actuator name="junior_car_motor_5double">
-                <hardwareInterface>VelocityJointInterface</hardwareInterface>
-                <mechanicalReduction>1</mechanicalReduction>
-            </actuator>
-        </transmission>  -->
-   <!-->  <transmission name="junior_car_tran_6double">
-            <robotNamespace>/junior_car</robotNamespace>
-            <type>transmission_interface/SimpleTransmission</type>
-            <joint name="left_drive_wheel_joint">
-                <hardwareInterface>VelocityJointInterface</hardwareInterface>
-            </joint>
-            <actuator name="junior_car_motor_6double">
-                <hardwareInterface>VelocityJointInterface</hardwareInterface>
-                <mechanicalReduction>1</mechanicalReduction>
-            </actuator>
-        </transmission> -->
     </xacro:macro>
 </robot>

File: box_sim/urdf/box.urdf.xacro (robot description, xacro)
@@ -1,183 +1,183 @@
 <?xml version="1.0"?>
 <robot name="box"
-  xmlns:xacro="http://www.ros.org/wiki/xacro">
-  <xacro:include filename="$(find box_sim)/urdf/box.gazebo.xacro" />
+    xmlns:xacro="http://www.ros.org/wiki/xacro">
+    <xacro:include filename="$(find box_sim)/urdf/box.gazebo.xacro" />
     <xacro:include filename="$(find box_sim)/urdf/box.transmission.xacro" />
-  <link name="base_link">
-    <inertial>
-      <origin xyz="0 0 0" rpy="0 0 0" />
-      <mass value="4.83" />
-      <inertia ixx="0" ixy="0" ixz="0" iyy="0" iyz="0" izz="0" />
-    </inertial>
-    <visual>
-      <origin xyz="0 0 0" rpy="0 0 0" />
-      <geometry>
-        <box size="1 0.6 0.25" />
-      </geometry>
-    </visual>
-  <collision>
-    <origin xyz="0 0 0" rpy="0 0 0" />
-      <geometry>
-         <box size="1 0.6 0.25" />
-      </geometry>
-    </collision>
-  </link>
-  <link name="right_steer_wheel_link">
-    <inertial>
-      <origin xyz="0 0 0" rpy="0 0 0" />
-      <mass value="0.9" />
-      <inertia ixx="0" ixy="0" ixz="0" iyy="0" iyz="0" izz="0" />
-    </inertial>
-    <visual>
-      <origin xyz="0 0 0" rpy="0 0 0" />
-      <geometry>
-        <cylinder length="0.1"  radius="0.1" />
-      </geometry>
-    </visual>
-  <collision>
-    <origin xyz="0 0 0" rpy="0 0 0" />
-      <geometry>
-        <cylinder length="0.1"  radius="0.1" />
-      </geometry>
-    </collision>
-  </link>
-  <joint name="right_steer_wheel_joint" type="continuous">
-    <origin xyz="0.40 -0.25 -0.25" rpy="0 1.5709 1.5709" />
-    <parent link="base_link" />
-    <child link="right_steer_wheel_link" />
-    <axis xyz = "0 0 1"/>
-  </joint>
+    <link name="base_link">
+        <inertial>
+            <origin xyz="0 0 0" rpy="0 0 0" />
+            <mass value="4.83" />
+            <inertia ixx="0" ixy="0" ixz="0" iyy="0" iyz="0" izz="0" />
+        </inertial>
+        <visual>
+            <origin xyz="0 0 0" rpy="0 0 0" />
+            <geometry>
+                <box size="1 0.6 0.25" />
+            </geometry>
+        </visual>
+        <collision>
+            <origin xyz="0 0 0" rpy="0 0 0" />
+            <geometry>
+                <box size="1 0.6 0.25" />
+            </geometry>
+        </collision>
+    </link>
+    <link name="right_steer_wheel_link">
+        <inertial>
+            <origin xyz="0 0 0" rpy="0 0 0" />
+            <mass value="0.9" />
+            <inertia ixx="0" ixy="0" ixz="0" iyy="0" iyz="0" izz="0" />
+        </inertial>
+        <visual>
+            <origin xyz="0 0 0" rpy="0 0 0" />
+            <geometry>
+                <cylinder length="0.1"  radius="0.1" />
+            </geometry>
+        </visual>
+        <collision>
+            <origin xyz="0 0 0" rpy="0 0 0" />
+            <geometry>
+                <cylinder length="0.1"  radius="0.1" />
+            </geometry>
+        </collision>
+    </link>
+    <joint name="right_steer_wheel_joint" type="continuous">
+        <origin xyz="0.40 -0.25 -0.25" rpy="0 1.5709 1.5709" />
+        <parent link="base_link" />
+        <child link="right_steer_wheel_link" />
+        <axis xyz = "0 0 1"/>
+    </joint>
     <link name="left_steer_wheel_link">
-    <inertial>
-      <origin xyz="0 0 0" rpy="0 0 0" />
-      <mass value="0.9" />
-      <inertia ixx="0" ixy="0" ixz="0" iyy="0" iyz="0" izz="0" />
-    </inertial>
-    <visual>
-      <origin xyz="0 0 0" rpy="0 0 0" />
-      <geometry>
-        <cylinder length="0.1"  radius="0.1" />
-      </geometry>
-    </visual>
-      <collision>
-    <origin xyz="0 0 0" rpy="0 0 0" />
-      <geometry>
-        <cylinder length="0.1"  radius="0.1" />
-      </geometry>
-    </collision>
-  </link>
-  <joint name="left_steer_wheel_joint" type="continuous">
-    <origin xyz="0.40 0.25 -0.25" rpy="0 1.5709 1.5709" />
-    <parent link="base_link" />
-    <child link="left_steer_wheel_link" />
-    <axis xyz = "0 0 1"/>
-  </joint>
+        <inertial>
+            <origin xyz="0 0 0" rpy="0 0 0" />
+            <mass value="0.9" />
+            <inertia ixx="0" ixy="0" ixz="0" iyy="0" iyz="0" izz="0" />
+        </inertial>
+        <visual>
+            <origin xyz="0 0 0" rpy="0 0 0" />
+            <geometry>
+                <cylinder length="0.1"  radius="0.1" />
+            </geometry>
+        </visual>
+        <collision>
+            <origin xyz="0 0 0" rpy="0 0 0" />
+            <geometry>
+                <cylinder length="0.1"  radius="0.1" />
+            </geometry>
+        </collision>
+    </link>
+    <joint name="left_steer_wheel_joint" type="continuous">
+        <origin xyz="0.40 0.25 -0.25" rpy="0 1.5709 1.5709" />
+        <parent link="base_link" />
+        <child link="left_steer_wheel_link" />
+        <axis xyz = "0 0 1"/>
+    </joint>
     <link name="right_drive_wheel_link">
-    <inertial>
-      <origin xyz="0 0 0" rpy="0 0 0" />
-      <mass value="0.9" />
-      <inertia ixx="0" ixy="0" ixz="0" iyy="0" iyz="0" izz="0" />
-    </inertial>
-    <visual>
-      <origin xyz="0 0 0" rpy="0 0 0" />
-      <geometry>
-        <cylinder length="0.1"  radius="0.1" />
-      </geometry>
-    </visual>
-      <collision>
-    <origin xyz="0 0 0" rpy="0 0 0" />
-      <geometry>
-        <cylinder length="0.1"  radius="0.1" />
-      </geometry>
-    </collision>
-  </link>
-  <joint name="right_drive_wheel_joint" type="continuous">
-    <origin xyz="-0.40 -0.25 -0.25" rpy="0 1.5709 1.5709" />
-    <parent link="base_link" />
-    <child link="right_drive_wheel_link" />
-    <axis xyz = "0 0 1"/>
-  </joint>
+        <inertial>
+            <origin xyz="0 0 0" rpy="0 0 0" />
+            <mass value="0.9" />
+            <inertia ixx="0" ixy="0" ixz="0" iyy="0" iyz="0" izz="0" />
+        </inertial>
+        <visual>
+            <origin xyz="0 0 0" rpy="0 0 0" />
+            <geometry>
+                <cylinder length="0.1"  radius="0.1" />
+            </geometry>
+        </visual>
+        <collision>
+            <origin xyz="0 0 0" rpy="0 0 0" />
+            <geometry>
+                <cylinder length="0.1"  radius="0.1" />
+            </geometry>
+        </collision>
+    </link>
+    <joint name="right_drive_wheel_joint" type="continuous">
+        <origin xyz="-0.40 -0.25 -0.25" rpy="0 1.5709 1.5709" />
+        <parent link="base_link" />
+        <child link="right_drive_wheel_link" />
+        <axis xyz = "0 0 1"/>
+    </joint>
     <link name="left_drive_wheel_link">
-    <inertial>
-      <origin xyz="0 0 0" rpy="0 0 0" />
-      <mass value="0.9" />
-      <inertia ixx="0" ixy="0" ixz="0" iyy="0" iyz="0" izz="0" />
-    </inertial>
-    <visual>
-      <origin xyz="0 0 0" rpy="0 0 0" />
-      <geometry>
-        <cylinder length="0.1"  radius="0.1" />
-      </geometry>
-    </visual>
-      <collision>
-    <origin xyz="0 0 0" rpy="0 0 0" />
-      <geometry>
-        <cylinder length="0.1"  radius="0.1" />
-      </geometry>
-    </collision>
-  </link>
-  <joint name="left_drive_wheel_joint" type="continuous">
-    <origin xyz="-0.40 0.25 -0.25" rpy="0 1.5709 1.5709" />
-    <parent link="base_link" />
-    <child link="left_drive_wheel_link" />
-    <axis xyz = "0 0 1"/>
-  </joint>
-  <link name="right_steer_link">
-    <inertial>
-      <origin xyz="0 0 0" rpy="0 0 0" />
-      <mass value="0.1" />
-      <inertia ixx="0" ixy="0" ixz="0" iyy="0" iyz="0" izz="0" />
-    </inertial>
-  </link>
-  <joint name="right_steer_joint" type="revolute">
-    <origin xyz="0.40 -0.25 -0.10" rpy="0 1.5709 1.5709" />
-    <parent link="base_link" />
-    <child link="right_steer_link" />
-    <axis xyz = "-1 0 0"/>
-    <dynamics damping="0.7" friction="0.7"/>
-    <limit effort="7.0" lower="-0.52" upper="0.52" velocity="${200.0*pi/180.0*0.95}"/>
-  </joint>
- <link name="left_steer_link">
-    <inertial>
-      <origin xyz="0 0 0" rpy="0 0 0" />
-      <mass value="0.9" />
-      <inertia ixx="0" ixy="0" ixz="0" iyy="0" iyz="0" izz="0" />
-    </inertial>
-  </link>
-  <joint name="left_steer_joint" type="revolute">
-    <origin xyz="0.40 0.25 -0.10" rpy="0 1.5709 1.5709" />
-    <parent link="base_link" />
-    <child link="left_steer_link" />
-    <dynamics damping="0.7" friction="0.7"/>
-    <limit effort="7.0" lower="-0.52" upper="0.52" velocity="${200.0*pi/180.0*0.95}"/>
-    <axis xyz = "-1 0 0"/>
-  </joint>
- <link name="fake_steer_link">
-    <inertial>
-      <origin xyz="0 0 0" rpy="0 0 0" />
-      <mass value="0.9" />
-      <inertia ixx="0" ixy="0" ixz="0" iyy="0" iyz="0" izz="0" />
-    </inertial>
-  </link>
-  <joint name="fake_steer_joint" type="revolute">
-    <origin xyz="0.40 0 -0.10" rpy="0 1.5709 1.5709" />
-    <parent link="base_link" />
-    <child link="fake_steer_link" />
-    <dynamics damping="0.7" friction="0.7"/>
-    <limit effort="7.0" lower="-0.52" upper="0.52" velocity="${200.0*pi/180.0*0.95}"/>
-    <axis xyz = "-1 0 0"/>
-  </joint>
-   <link name="fake_drive_link">
-    <inertial>
-      <origin xyz="0 0 0" rpy="0 0 0" />
-      <mass value="0.9" />
-      <inertia ixx="0" ixy="0" ixz="0" iyy="0" iyz="0" izz="0" />
-    </inertial>
-  </link>
-  <joint name="fake_drive_joint" type="continuous">
-    <origin xyz="-0.40 0 -0.25" rpy="0 1.5709 1.5709" />
-    <parent link="base_link" />
-    <child link="fake_drive_link" />
-    <axis xyz = "0 0 1"/>
-  </joint>
+        <inertial>
+            <origin xyz="0 0 0" rpy="0 0 0" />
+            <mass value="0.9" />
+            <inertia ixx="0" ixy="0" ixz="0" iyy="0" iyz="0" izz="0" />
+        </inertial>
+        <visual>
+            <origin xyz="0 0 0" rpy="0 0 0" />
+            <geometry>
+                <cylinder length="0.1"  radius="0.1" />
+            </geometry>
+        </visual>
+        <collision>
+            <origin xyz="0 0 0" rpy="0 0 0" />
+            <geometry>
+                <cylinder length="0.1"  radius="0.1" />
+            </geometry>
+        </collision>
+    </link>
+    <joint name="left_drive_wheel_joint" type="continuous">
+        <origin xyz="-0.40 0.25 -0.25" rpy="0 1.5709 1.5709" />
+        <parent link="base_link" />
+        <child link="left_drive_wheel_link" />
+        <axis xyz = "0 0 1"/>
+    </joint>
+    <link name="right_steer_link">
+        <inertial>
+            <origin xyz="0 0 0" rpy="0 0 0" />
+            <mass value="0.1" />
+            <inertia ixx="0" ixy="0" ixz="0" iyy="0" iyz="0" izz="0" />
+        </inertial>
+    </link>
+    <joint name="right_steer_joint" type="revolute">
+        <origin xyz="0.40 -0.25 -0.10" rpy="0 1.5709 1.5709" />
+        <parent link="base_link" />
+        <child link="right_steer_link" />
+        <axis xyz = "-1 0 0"/>
+        <dynamics damping="0.7" friction="0.7"/>
+        <limit effort="7.0" lower="-0.52" upper="0.52" velocity="${200.0*pi/180.0*0.95}"/>
+    </joint>
+    <link name="left_steer_link">
+        <inertial>
+            <origin xyz="0 0 0" rpy="0 0 0" />
+            <mass value="0.9" />
+            <inertia ixx="0" ixy="0" ixz="0" iyy="0" iyz="0" izz="0" />
+        </inertial>
+    </link>
+    <joint name="left_steer_joint" type="revolute">
+        <origin xyz="0.40 0.25 -0.10" rpy="0 1.5709 1.5709" />
+        <parent link="base_link" />
+        <child link="left_steer_link" />
+        <dynamics damping="0.7" friction="0.7"/>
+        <limit effort="7.0" lower="-0.52" upper="0.52" velocity="${200.0*pi/180.0*0.95}"/>
+        <axis xyz = "-1 0 0"/>
+    </joint>
+    <link name="fake_steer_link">
+        <inertial>
+            <origin xyz="0 0 0" rpy="0 0 0" />
+            <mass value="0.9" />
+            <inertia ixx="0" ixy="0" ixz="0" iyy="0" iyz="0" izz="0" />
+        </inertial>
+    </link>
+    <joint name="fake_steer_joint" type="revolute">
+        <origin xyz="0.40 0 -0.10" rpy="0 1.5709 1.5709" />
+        <parent link="base_link" />
+        <child link="fake_steer_link" />
+        <dynamics damping="0.7" friction="0.7"/>
+        <limit effort="7.0" lower="-0.52" upper="0.52" velocity="${200.0*pi/180.0*0.95}"/>
+        <axis xyz = "-1 0 0"/>
+    </joint>
+    <link name="fake_drive_link">
+        <inertial>
+            <origin xyz="0 0 0" rpy="0 0 0" />
+            <mass value="0.9" />
+            <inertia ixx="0" ixy="0" ixz="0" iyy="0" iyz="0" izz="0" />
+        </inertial>
+    </link>
+    <joint name="fake_drive_joint" type="continuous">
+        <origin xyz="-0.40 0 -0.25" rpy="0 1.5709 1.5709" />
+        <parent link="base_link" />
+        <child link="fake_drive_link" />
+        <axis xyz = "0 0 1"/>
+    </joint>
 </robot>
